Commit message: Create fishbot URDF with modular sensor components
- Reorganize sensor files and base URDF into fishbot folder
- Create fishbot.urdf.xacro that includes and instantiates sensor macros
- Define base_link with cylinder (length=0.12, radius=0.1)
- Mount IMU at (0, 0, 0.02), camera at (0.1, 0, 0.075), laser at (0, 0, 0.12)
- Update sensor macros to work with new folder structure

Co-authored-by: Copilot <223556219+Copilot@users.noreply.github.com>

File: src/mybot_description/urdf/fishbot/sensor/camera.urdf.xacro (robot description, xacro)
@@ -1,8 +1,8 @@
 <?xml version="1.0"?>
 <robot xmlns:xacro="http://www.ros.org/wiki/xacro">
-    <xacro:macro name="camera_xacro" params = "joint_xyz link_xyz">
-        <link name="${camera_name}_link">
+    <xacro:macro name="camera_xacro" params = "joint_xyz">
+        <link name="camera_link">
             <visual>
-                <origin xyz="${link_xyz}" rpy="0 0 0"/>
+                <origin xyz="0 0 0" rpy="0 0 0"/>
                 <geometry>
                     <box size="0.02 0.02 0.02"/>
@@ -15,5 +15,5 @@
         <joint name="camera_joint" type="fixed">
             <parent link="base_link"/>
-            <child link="${camera_name}_link"/>
+            <child link="camera_link"/>
             <origin xyz="${joint_xyz}" rpy="0 0 0"/>
         </joint>

File: src/mybot_description/urdf/fishbot/sensor/imu.urdf.xacro (robot description, xacro)
@@ -4,8 +4,8 @@
   <xacro:include filename="$(find mybot_description)/urdf/first_robot_arm.xacro"/>
   <xacro:include filename="$(find mybot_description)/urdf/first_robot_gripper.xacro"/> -->
-    <xacro:macro name="imu_xacro" params = "joint_xyz link_xyz">
-        <link name="${imu_name}_link">
+    <xacro:macro name="imu_xacro" params = "joint_xyz">
+        <link name="imu_link">
             <visual>
-                <origin xyz="${link_xyz}" rpy="0 0 0"/>
+                <origin xyz="0 0 0" rpy="0 0 0"/>
                 <geometry>
                     <box size="0.02 0.02 0.02"/>
@@ -18,5 +18,5 @@
         <joint name="imu_joint" type="fixed">
             <parent link="base_link"/>
-            <child link="${imu_name}_link"/>
+            <child link="$imu_link"/>
             <origin xyz="${joint_xyz}" rpy="0 0 0"/>
         </joint>
