Commit message: feat: complete FishBot sensor URDF and add workspace documentation
URDF fixes:
- Add missing <inertial> tags to all sensor links for Gazebo compatibility
  - imu_link, camera_link, laser_link (0.01 kg each)
  - laser_support_link (0.05 kg, cylinder inertia)
- Fix typo in imu.urdf.xacro: $imu_link -> imu_link

Documentation:
- Rewrite README.md with complete workspace overview
- Document all 5 packages (interface, mybot_description, my_cpp_pkg, my_py_pkg, wpr_simulation2)
- Add FishBot model structure and quick start commands

File: src/mybot_description/urdf/fishbot/sensor/camera.urdf.xacro (robot description, xacro)
@@ -12,4 +12,9 @@
                 </material>
             </visual>
+            <inertial>
+                <origin xyz="0 0 0" rpy="0 0 0"/>
+                <mass value="0.01"/>
+                <inertia ixx="3.33e-6" ixy="0" ixz="0" iyy="3.33e-6" iyz="0" izz="3.33e-6"/>
+            </inertial>
         </link>
         <joint name="camera_joint" type="fixed">

File: src/mybot_description/urdf/fishbot/sensor/imu.urdf.xacro (robot description, xacro)
@@ -15,8 +15,13 @@
                 </material>
             </visual>
+            <inertial>
+                <origin xyz="0 0 0" rpy="0 0 0"/>
+                <mass value="0.01"/>
+                <inertia ixx="3.33e-6" ixy="0" ixz="0" iyy="3.33e-6" iyz="0" izz="3.33e-6"/>
+            </inertial>
         </link>
         <joint name="imu_joint" type="fixed">
             <parent link="base_link"/>
-            <child link="$imu_link"/>
+            <child link="imu_link"/>
             <origin xyz="${joint_xyz}" rpy="0 0 0"/>
         </joint>

File: src/mybot_description/urdf/fishbot/sensor/laser.urdf.xacro (robot description, xacro)
@@ -13,4 +13,9 @@
                 </material>
             </visual>
+            <inertial>
+                <origin xyz="0 0 0" rpy="0 0 0"/>
+                <mass value="0.05"/>
+                <inertia ixx="4.58e-5" ixy="0" ixz="0" iyy="4.58e-5" iyz="0" izz="2.5e-6"/>
+            </inertial>
         </link>
         <!-- 支撑杆与 base_link 的关节 -->
@@ -31,4 +36,9 @@
                 </material>
             </visual>
+            <inertial>
+                <origin xyz="0 0 0" rpy="0 0 0"/>
+                <mass value="0.01"/>
+                <inertia ixx="3.33e-6" ixy="0" ixz="0" iyy="3.33e-6" iyz="0" izz="3.33e-6"/>
+            </inertial>
         </link>
         <!-- 雷达与支撑杆的关节 -->
