Commit message: 修改fishbot的urdf文件

File: src/mybot_description/urdf/fishbot/base.urdf.xacro (robot description, xacro)
@@ -5,18 +5,26 @@
   <xacro:include filename="$(find mybot_description)/urdf/first_robot_gripper.xacro"/> -->
     <xacro:macro name="base_xacro" params="length radius">
-            <!--机器人身体-->
+        <!--机器人底盘-->
         <link name="base_link">
+            <inertial>
+                <mass value="2.0"/>
+                <origin xyz="0 0 0" rpy="0 0 0"/>
+                <inertia ixx="0.1" ixy="0.0" ixz="0.0" iyy="0.1" iyz="0.0" izz="0.1"/>
+            </inertial>
             <visual>
-                <!--沿自己几何中心偏移量-->
-                <origin xyz="0 0 0.0" rpy="0 0 0"/>
-                <!--几何形状-->
+                <origin xyz="0 0 0" rpy="0 0 0"/>
                 <geometry>
                     <cylinder radius="${radius}" length="${length}"/>
                 </geometry>
-                <!--材质和颜色-->
-                <material name="white">
-                    <color rgba="1 1 1 0.5"/>
+                <material name="blue">
+                    <color rgba="0 0 0 0.5"/>
                 </material>
             </visual>
+            <collision>
+                <origin xyz="0 0 0" rpy="0 0 0"/>
+                <geometry>
+                    <cylinder radius="${radius}" length="${length}"/>
+                </geometry>
+            </collision>
         </link>
     </xacro:macro>

File: src/mybot_description/urdf/fishbot/fishbot.urdf.xacro (robot description, xacro)
@@ -1,29 +1,12 @@
 <?xml version="1.0"?>
 <robot name="fishbot" xmlns:xacro="http://www.ros.org/wiki/xacro">
+  <!-- Include base macro -->
+  <xacro:include filename="$(find mybot_description)/urdf/fishbot/base.urdf.xacro"/>
   <!-- Include modular sensor components from sensor folder -->
   <xacro:include filename="$(find mybot_description)/urdf/fishbot/sensor/camera.urdf.xacro"/>
   <xacro:include filename="$(find mybot_description)/urdf/fishbot/sensor/imu.urdf.xacro"/>
   <xacro:include filename="$(find mybot_description)/urdf/fishbot/sensor/laser.urdf.xacro"/>
-  <!-- Base link: cylinder length=0.12, radius=0.1 -->
-  <link name="base_link">
-    <inertial>
-      <mass value="2.0"/>
-      <origin xyz="0 0 0" rpy="0 0 0"/>
-      <inertia ixx="0.1" ixy="0.0" ixz="0.0" iyy="0.1" iyz="0.0" izz="0.1"/>
-    </inertial>
-    <visual>
-      <geometry>
-        <cylinder length="0.12" radius="0.1"/>
-      </geometry>
-      <origin xyz="0 0 0" rpy="0 0 0"/>
-      <material name="blue"><color rgba="0 0.5 1 1"/></material>
-    </visual>
-    <collision>
-      <geometry>
-        <cylinder length="0.12" radius="0.1"/>
-      </geometry>
-      <origin xyz="0 0 0" rpy="0 0 0"/>
-    </collision>
-  </link>
+  <!-- Instantiate base: cylinder length=0.12, radius=0.1 -->
+  <xacro:base_xacro length="0.12" radius="0.1"/>
   <!-- Instantiate sensors with provided parameters -->
   <xacro:imu_xacro joint_xyz="0 0 0.02"/>

Commit message: 5月18日  18：50

File: src/mybot_description/urdf/fishbot/base.urdf.xacro (robot description, xacro)
@@ -10,5 +10,5 @@
                 <mass value="2.0"/>
                 <origin xyz="0 0 0" rpy="0 0 0"/>
-                <inertia ixx="0.1" ixy="0.0" ixz="0.0" iyy="0.1" iyz="0.0" izz="0.1"/>
+                <inertia ixx="0.0117" ixy="0.0" ixz="0.0" iyy="0.0117" iyz="0.0" izz="0.01"/>
             </inertial>
             <visual>
@@ -28,4 +28,12 @@
             </collision>
         </link>
+        <link name="base_footprint_link">
+        </link>
+        <!--底盘与足迹链接-->
+        <joint name="base_to_footprint" type="fixed">
+            <parent link="base_footprint_link"/>
+            <child link="base_link"/>
+            <origin xyz="0 0 ${length/2+0.031}" rpy="0 0 0"/>
+        </joint>
     </xacro:macro>
 </robot>

File: src/mybot_description/urdf/fishbot/fishbot.urdf.xacro (robot description, xacro)
@@ -7,9 +7,15 @@
   <xacro:include filename="$(find mybot_description)/urdf/fishbot/sensor/imu.urdf.xacro"/>
   <xacro:include filename="$(find mybot_description)/urdf/fishbot/sensor/laser.urdf.xacro"/>
+  <xacro:include filename="$(find mybot_description)/urdf/fishbot/actuator/wheel.xacro"/>
+  <xacro:include filename="$(find mybot_description)/urdf/fishbot/actuator/caster.xacro"/>
   <!-- Instantiate base: cylinder length=0.12, radius=0.1 -->
-  <xacro:base_xacro length="0.12" radius="0.1"/>
+  <xacro:base_xacro length="0.1" radius="0.12"/>
   <!-- Instantiate sensors with provided parameters -->
   <xacro:imu_xacro joint_xyz="0 0 0.02"/>
-  <xacro:camera_xacro joint_xyz="0.1 0 0.075"/>
-  <xacro:laser_xacro joint_xyz="0 0 0.12"/>
+  <xacro:camera_xacro joint_xyz="0.1 0 0.05"/>
+  <xacro:laser_xacro joint_xyz="0 0 0.1"/>
+  <xacro:wheel_xacro wheel_name="left_wheel" xyz="0 0.1 -0.05"/>
+  <xacro:wheel_xacro wheel_name="right_wheel" xyz="0 -0.1 -0.05"/>
+  <xacro:caster_xacro caster_name="front_caster" xyz="0.08 0 -0.05"/>
+  <xacro:caster_xacro caster_name="back_caster" xyz="-0.08 0 -0.05"/>
 </robot>

File: src/mybot_description/urdf/fishbot/sensor/laser.urdf.xacro (robot description, xacro)
@@ -13,4 +13,10 @@
                 </material>
             </visual>
+            <collision>
+                <origin xyz="0 0 0" rpy="0 0 0"/>
+                <geometry>
+                    <cylinder radius="0.01" length="0.1"/>
+                </geometry>
+            </collision>
             <inertial>
                 <origin xyz="0 0 0" rpy="0 0 0"/>
@@ -36,4 +42,10 @@
                 </material>
             </visual>
+            <collision>
+                <origin xyz="0 0 0" rpy="0 0 0"/>
+                <geometry>
+                    <box size="0.02 0.02 0.02"/>
+                </geometry>
+            </collision>
             <inertial>
                 <origin xyz="0 0 0" rpy="0 0 0"/>
