Commit message: 5月19日 16：47

File: src/mybot_description/urdf/fishbot/actuator/caster.xacro (robot description, xacro)
@@ -31,4 +31,13 @@
       </collision>
     </link>
+    <gazebo reference="${caster_name}_link">
+      <material>Gazebo/Black</material>
+    </gazebo>
+    <gazebo reference="${caster_name}_link">
+      <mu>0.0</mu>
+      <mu2>0.0</mu2>
+      <kp>1000000.0</kp>
+      <kd>1.0</kd>
+    </gazebo>
   </xacro:macro>
 </robot>

File: src/mybot_description/urdf/fishbot/actuator/wheel.xacro (robot description, xacro)
@@ -32,4 +32,14 @@
       </collision>
     </link>
+    <gazebo reference="${wheel_name}_link">
+      <material>Gazebo/Black</material>
+    </gazebo>
+    <!-- 轮子物理属性 -->
+    <gazebo reference="${wheel_name}_link">
+      <mu>20.0</mu>
+      <mu2>20.0</mu2>
+      <kp>1000000.0</kp>
+      <kd>1.0</kd>
+    </gazebo>
   </xacro:macro>
 </robot>

File: src/mybot_description/urdf/fishbot/base.urdf.xacro (robot description, xacro)
@@ -28,4 +28,7 @@
             </collision>
         </link>
+        <gazebo reference="base_link">
+            <material>Gazebo/Blue</material>
+        </gazebo>
         <link name="base_footprint_link">
         </link>

File: src/mybot_description/urdf/fishbot/fishbot.urdf.xacro (robot description, xacro)
@@ -9,4 +9,7 @@
   <xacro:include filename="$(find mybot_description)/urdf/fishbot/actuator/wheel.xacro"/>
   <xacro:include filename="$(find mybot_description)/urdf/fishbot/actuator/caster.xacro"/>
+  <xacro:include filename="$(find mybot_description)/urdf/fishbot/plugins/gazebo_control_plugins.xacro"/>
+  <xacro:include filename="$(find mybot_description)/urdf/fishbot/plugins/gazebo_sensor_plugins.xacro"/>
+   <!-- Instantiate Gazebo control plugins -->
   <!-- Instantiate base: cylinder length=0.12, radius=0.1 -->
   <xacro:base_xacro length="0.1" radius="0.12"/>
@@ -19,3 +22,5 @@
   <xacro:caster_xacro caster_name="front_caster" xyz="0.08 0 -0.05"/>
   <xacro:caster_xacro caster_name="back_caster" xyz="-0.08 0 -0.05"/>
+  <xacro:gazebo_control_plugins/>
+  <xacro:gazebo_sensor_plugin/>
 </robot>

File: src/mybot_description/urdf/fishbot/sensor/camera.urdf.xacro (robot description, xacro)
@@ -18,4 +18,7 @@
             </inertial>
         </link>
+        <gazebo reference="camera_link">
+            <material>Gazebo/Red</material>
+        </gazebo>
         <joint name="camera_joint" type="fixed">
             <parent link="base_link"/>

File: src/mybot_description/urdf/fishbot/sensor/imu.urdf.xacro (robot description, xacro)
@@ -21,4 +21,7 @@
             </inertial>
         </link>
+        <gazebo reference="imu_link">
+            <material>Gazebo/Red</material>
+        </gazebo>
         <joint name="imu_joint" type="fixed">
             <parent link="base_link"/>

File: src/mybot_description/urdf/fishbot/sensor/laser.urdf.xacro (robot description, xacro)
@@ -25,4 +25,7 @@
             </inertial>
         </link>
+        <gazebo reference="laser_support_link">
+            <material>Gazebo/Black</material>
+        </gazebo>
         <!-- 支撑杆与 base_link 的关节 -->
         <joint name="laser_support_joint" type="fixed">
@@ -54,4 +57,7 @@
             </inertial>
         </link>
+        <gazebo reference="laser_link">
+            <material>Gazebo/Red</material>
+        </gazebo>
         <!-- 雷达与支撑杆的关节 -->
         <joint name="laser_joint" type="fixed">
