Commit message: feat: gazebo imu & depth camera plugins

File: src/mybot_description/urdf/fishbot/plugins/gazebo_sensor_plugins.xacro (robot description, xacro)
@@ -2,4 +2,5 @@
 <robot xmlns:xacro="http://www.ros.org/wiki/xacro">
     <xacro:macro name="gazebo_sensor_plugin">
+        <!-- 激光雷达传感器插件 -->
         <gazebo reference="laser_link">
             <sensor type="ray" name="laserscan">
@@ -38,4 +39,90 @@
             </sensor>
         </gazebo>
+        <!-- IMU传感器插件 -->
+        <gazebo reference="imu_link">
+            <sensor type="imu" name="imu_sensor">
+                <plugin name="gazebo_ros_imu_controller" filename="libgazebo_ros_imu_sensor.so">
+                    <ros>
+                        <namespace>/</namespace>
+                        <remapping>~/out:=/imu</remapping>
+                    </ros>
+                    <frame_name>imu_link</frame_name>
+                    <initial_orientation_as_reference>false</initial_orientation_as_reference>
+                </plugin>
+                <always_on>true</always_on>
+                <update_rate>100.0</update_rate>
+                <visualize>true</visualize>
+                <imu>
+                    <angular_velocity>
+                        <x>
+                            <noise type="gaussian">
+                                <mean>0.0</mean>
+                                <stddev>0.001</stddev>
+                            </noise>
+                        </x>
+                        <y>
+                            <noise type="gaussian">
+                                <mean>0.0</mean>
+                                <stddev>0.001</stddev>
+                            </noise>
+                        </y>
+                        <z>
+                            <noise type="gaussian">
+                                <mean>0.0</mean>
+                                <stddev>0.001</stddev>
+                            </noise>
+                        </z>
+                    </angular_velocity>
+                    <linear_acceleration>
+                        <x>
+                            <noise type="gaussian">
+                                <mean>0.0</mean>
+                                <stddev>0.01</stddev>
+                            </noise>
+                        </x>
+                        <y>
+                            <noise type="gaussian">
+                                <mean>0.0</mean>
+                                <stddev>0.01</stddev>
+                            </noise>
+                        </y>
+                        <z>
+                            <noise type="gaussian">
+                                <mean>0.0</mean>
+                                <stddev>0.01</stddev>
+                            </noise>
+                        </z>
+                    </linear_acceleration>
+                </imu>
+            </sensor>
+        </gazebo>
+        <!-- 相机传感器插件 -->
+        <gazebo reference="camera_link">
+            <sensor type="depth" name="depth_camera_sensor">
+                <plugin name="gazebo_ros_depth_camera_controller" filename="libgazebo_ros_camera.so">
+                    <frame_name>camera_optical_link</frame_name>
+                </plugin>
+                <always_on>true</always_on>
+                <update_rate>30.0</update_rate>
+                <visualize>true</visualize>
+                <camera>
+                    <horizontal_fov>1.047</horizontal_fov>
+                    <image>
+                        <width>640</width>
+                        <height>480</height>
+                        <format>R8G8B8</format>
+                    </image>
+                    <clip>
+                        <near>0.05</near>
+                        <far>10</far>
+                    </clip>
+                    <noise>
+                        <type>gaussian</type>
+                        <mean>0.0</mean>
+                        <stddev>0.007</stddev>
+                    </noise>
+                </camera>
+            </sensor>
+        </gazebo>
     </xacro:macro>
 </robot>

File: src/mybot_description/urdf/fishbot/sensor/camera.urdf.xacro (robot description, xacro)
@@ -2,4 +2,5 @@
 <robot xmlns:xacro="http://www.ros.org/wiki/xacro">
     <xacro:macro name="camera_xacro" params = "joint_xyz">
+        <!-- 相机本体 -->
         <link name="camera_link">
             <visual>
@@ -18,4 +19,6 @@
             </inertial>
         </link>
+        <!-- 相机旋转虚拟部件 -->
+        <link name="camera_optical_link"></link>
         <gazebo reference="camera_link">
             <material>Gazebo/Red</material>
@@ -26,4 +29,9 @@
             <origin xyz="${joint_xyz}" rpy="0 0 0"/>
         </joint>
+        <joint name="camera_optical_joint" type="fixed">
+            <parent link="camera_link"/>
+            <child link="camera_optical_link"/>
+            <origin xyz="0 0 0" rpy="${-pi/2} 0 ${-pi/2}"/>
+        </joint>
     </xacro:macro>
 </robot>
